File: Pure VCO.sch (EAGLE design)
At the start: 76 parts, among them T1 TRANS_PAIR, T2 N_CHN, U1 QUAD_OPAMP, U2 QUAD_OPAMP, U3 DUAL_OPAMP

Commit message: VCO 2.1
Parts:
- R23: value 19K -> 19k1
- R35: value 15K -> 3K3
- R39: value 2K2 -> 100K
- R40: value 2K2 -> 2M
- R41: value 2K2 -> 3K3
- R42: value 2K2 -> 1K5
- TR1: device INSTRUO:TRIM_3269W -> INSTRUO:TRIMMER_TH3
- renumbered 2M to R40, 2M1 to R39, 2M2 to R37, 2M3 to R38, 2M4 to R41, 2M5 to R42, 3K1 to R36, 3K3 to R35

Commit message: VCO 2.3
Parts:
- removed 1V/OCT, LIN-FM, PULSE, PWM, SAW, SYNC, TRI: S_JACK, INSTRUO:S_JACK
- removed COARSE, FINE, FM_ATT, PWM_ATT, PWM_POT: B100K, INSTRUO:Q-POT
- removed R0: 2K, INSTRUO:R_TC
- removed T2: N_CHN, INSTRUO:N_CHN
- removed U2: QUAD_OPAMP, INSTRUO:QUAD_OPAMP
- removed U3: DUAL_OPAMP, INSTRUO:DUAL_OPAMP
- added C15, C16, C18, C19: 100n, GMSN:C-USC0805K
- added C17: 100p, GMSN:C-USC0805K
- added CP1, CP2: 10u, GMSN:CPOL-US153CLV-0505
- added IC1, IC2, IC3, IC4, IC5, IC6: TL072D, GMSN:TL072D
- added J1, J2, J3, J4, J5, J6, J7, J8: S_JACK, GMSN:S_JACK
- added R15: 56K, GMSN:R-US_R0805
- added R22: 1K5, GMSN:R-US_R0805
- added R29: 2K, GMSN:R-US_R0805
- added R3: 100K, GMSN:R-US_R0805
- added R43, R44, R46: 10K, GMSN:R-US_R0805
- added R45: empty, GMSN:R-US_R0805
- added R47: 1K3, GMSN:R-US_R0805
- added R6: 390R, GMSN:R-US_R0805
- added R7: 87k, GMSN:R-US_R0805
- added TC1: 2K, GMSN:R_TC
- added TP1, TP2: TRANS_PAIR, GMSN:TRANS_PAIR
- added TR4, TR5: 100K, GMSN:TRIMMER_TH3
- added VR1: Coarse, GMSN:9MMPOT
- added VR2, VR3, VR4, VR5: B100K, GMSN:9MMPOT
- C1, C2: value (none) -> 100n; device rcl:CPOL-US153CLV-0505 -> GMSN:C-USC0805K
- C10, C11, C12, C3, C9: device rcl:C-USC0805K -> GMSN:C-USC0805K
- C13: value 100n -> 10nF; device rcl:C-USC0805K -> GMSN:C-USC0805K
- C14: value 100n -> 1000p; device rcl:C-USC0805K -> GMSN:C-USC0805K
- C4: value 2.2n -> 100p; device INSTRUO:CAP_POLY -> GMSN:C-USC0805K
- C5: value 100p -> 100n; device rcl:C-USC0805K -> GMSN:C-USC0805K
- C6: value 22p -> 100n; device rcl:C-USC0805K -> GMSN:C-USC0805K
- C7: value 10nF -> 2.2n; device rcl:C-USC0805K -> GMSN:CAP_POLY
- C8: value 1000p -> 22p; device rcl:C-USC0805K -> GMSN:C-USC0805K
- D1, D2: device adafruit:DIODESMA -> GMSN:DIODESMA
- D3, D4: device SparkFun-DiscreteSemi:DIODESOD -> GMSN:DIODESOD-323F
- R1, R2: device rcl:R-US_R0805 -> GMSN:R-US_R0805
- R10: value 680R -> 39K; device rcl:R-US_R0805 -> GMSN:R-US_R0805
- R11: value 15K -> 680R; device rcl:R-US_R0805 -> GMSN:R-US_R0805
- R12: value 22K -> 9K1; device rcl:R-US_R0805 -> GMSN:R-US_R0805
- R13: value 10K -> 5K6; device rcl:R-US_R0805 -> GMSN:R-US_R0805
- R14: value 39K -> 10K; device rcl:R-US_R0805 -> GMSN:R-US_R0805
- R16: value 56K -> 100K; device rcl:R-US_R0805 -> GMSN:R-US_R0805
- R17: value 5K6 -> 39K; device rcl:R-US_R0805 -> GMSN:R-US_R0805
- R18: value 10K -> 2K2; device rcl:R-US_R0805 -> GMSN:R-US_R0805
- R19: value 10K -> 2M; device rcl:R-US_R0805 -> GMSN:R-US_R0805
- R20: value 22K* -> 10K; device rcl:R-US_R0805 -> GMSN:R-US_R0805
- R21: value 22K* -> 3K3; device rcl:R-US_R0805 -> GMSN:R-US_R0805
- R23: value 19k1 -> 10K; device rcl:R-US_R0805 -> GMSN:R-US_R0805
- R24, R25: value 2K -> 22K*; device rcl:R-US_R0805 -> GMSN:R-US_R0805
- R26: value 10K -> 19k1; device rcl:R-US_R0805 -> GMSN:R-US_R0805
- R27: value 100K -> 2K; device rcl:R-US_R0805 -> GMSN:R-US_R0805
- R28: value 27K -> 10K; device rcl:R-US_R0805 -> GMSN:R-US_R0805
- R30: value * -> 100K; device rcl:R-US_R0805 -> GMSN:R-US_R0805
- R31: value 10K -> 27K; device rcl:R-US_R0805 -> GMSN:R-US_R0805
- R32: value 1K3 -> 10K; device rcl:R-US_R0805 -> GMSN:R-US_R0805
- R33: value 2K -> 1K3; device rcl:R-US_R0805 -> GMSN:R-US_R0805
- R34: value 2K2 -> 2K; device rcl:R-US_R0805 -> GMSN:R-US_R0805
- R35: value 3K3 -> 1K3; device rcl:R-US_R0805 -> GMSN:R-US_R0805
- R36: value 9K1 -> 3K3; device rcl:R-US_R0805 -> GMSN:R-US_R0805
- R37: value 39K -> 2K; device rcl:R-US_R0805 -> GMSN:R-US_R0805
- R38: value 120K -> 10K; device rcl:R-US_R0805 -> GMSN:R-US_R0805
- R39: value 100K -> 402R; device rcl:R-US_R0805 -> GMSN:R-US_R0805
- R4: value 390R -> 2M; device rcl:R-US_R0805 -> GMSN:R-US_R0805
- R40: value 2M -> 10K; device rcl:R-US_R0805 -> GMSN:R-US_R0805
- R41: value 3K3 -> 10K; device rcl:R-US_R0805 -> GMSN:R-US_R0805
- R42: value 1K5 -> 2K; device rcl:R-US_R0805 -> GMSN:R-US_R0805
- R5: value 100K -> 560K; device rcl:R-US_R0805 -> GMSN:R-US_R0805
- R8: value 560K -> 3K3; device rcl:R-US_R0805 -> GMSN:R-US_R0805
- R9: value 2M -> 120K; device rcl:R-US_R0805 -> GMSN:R-US_R0805
- T1: value TRANS_PAIR -> N_CHN; device INSTRUO:TRANS_PAIR -> GMSN:N_CHN
- TR1: device INSTRUO:TRIMMER_TH3 -> GMSN:TRIMMER_TH3
- TR2, TR3: device INSTRUO:TRIM_3269W -> GMSN:TRIMMER_TH3
- U1: value QUAD_OPAMP -> LM4040A50IDBZT; device INSTRUO:QUAD_OPAMP -> GMSN:LM4040A50IDBZT
Connections:
- removed net N$25: C7.1, D3.A, R14.1, R20.2, R34.1, U2G$1.OUT
- removed net N$35: R30.2, U2G$3.+IN
- removed net N$38: R32.1, R33.1, TRI.TIP
- removed net N$43: R39.2, U3G$1.-IN, U3G$2.OUT
- removed net N$45: U2G$2.-IN, U2G$2.OUT
- new net N$14: C17.1, IC6A.-IN, R38.2, R44.2, TP2G$2.C
- new net N$6: IC3A.OUT, IC3B.-IN, R16.2
- new net N$75: IC5B.OUT, R47.1, TR4.1, TR4.2
- new net N$76: R37.1, TP2G$2.B, TR4.3
- new net N$77: R39.1, TP2G$2.E, TR5.1
- new net N$78: R39.2, TP2G$1.E, TR5.3
- new net N$79: R40.1, TR5.2
- new net N$80: R42.1, TP2G$1.B
- new net N$82: IC6A.+IN, R41.2, R43.1, TP2G$1.C
- new net N$83: IC5B.+IN, R35.1, R36.1
- new net N$84: IC6B.-IN, R45.2, R46.2
- new net PULSEIN: C13.1, D3.A, IC4A.OUT, R17.1, R18.1, R24.2
- new net SAWCORE: IC2A.OUT, R11.1, R12.1, R14.2
- new net SINE: IC6B.OUT, J8.TIP, R46.1
- new net SINE_PRE1: C17.2, IC6A.OUT, IC6B.+IN, R44.1
- new net TRI: J7.TIP, R33.1, R34.1, R35.2
- net +12V: now also C1.1, C15.1, C18.1, C5.1, CP1.+, IC1P.V+, IC2P.V+, IC3P.V+, IC4P.V+, IC5P.V+, IC6P.V+, R38.1, R4.2, R41.1, R7.2, VR1.3, VR2.3, VR4.3; no longer C1.+, C13.1, COARSE.3, FINE.3, PWM_POT.3, R12.2, R9.2, U1G$5.+12V, U2G$5.+12V, U3G$3.+12V
- net -12V: now also C16.2, C19.2, C2.2, C6.2, CP2.-, IC1P.V-, IC2P.V-, IC3P.V-, IC4P.V-, IC5P.V-, IC6P.V-, R15.2, R26.2, R31.1, R40.2, VR1.1, VR2.1, VR4.1; no longer C14.2, C2.-, COARSE.1, FINE.1, PWM_POT.1, R16.2, R23.2, R28.1, U1G$6.-12V, U2G$6.-12V, U3G$4.-12V
- net GND: now also C1.2, C15.2, C16.1, C18.2, C19.1, C2.1, C5.2, C6.1, CP1.-, CP2.+, IC1A.+IN, IC1B.+IN, IC2A.+IN, IC3A.+IN, IC4A.+IN, IC4B.+IN, IC5A.+IN, J1.GND, J1.NORM, J2.GND, J2.NORM, J3.GND, J4.GND, J5.GND, J6.GND, J7.GND, J8.GND, R20.2, R22.1, R29.2, R34.2, R36.2, R37.2, R42.2, R43.2, R45.1, R6.1, R8.1, TP1G$1.B, U1.ANODE, VR3.1, VR5.1; no longer 1V/OCT.GND, 1V/OCT.NORM, C1.-, C13.2, C14.1, C2.+, FM_ATT.1, LIN-FM.GND, LIN-FM.NORM, PULSE.GND, PWM.GND, PWM_ATT.1, R11.1, R18.2, R25.2, R30.1, R33.2, R35.1, R4.1, R42.1, SAW.GND, SYNC.GND, T1G$2.B, TRI.GND, U1G$1.+IN, U1G$2.+IN, U1G$4.+IN, U2G$1.+IN, U2G$2.+IN, U2G$4.+IN, U3G$2.+IN
- net N$10: now also TP1G$2.B; no longer T1G$1.B
- net N$11: now also C7.-, R11.2, T1.D; no longer C4.-, R10.2, T2.D
- net N$12: now also IC1B.-IN, R4.1, R5.1, TP1G$2.C; no longer R8.1, R9.1, T1G$1.C, U1G$4.-IN
- net N$13: now also C7.+, IC2A.-IN, T1.S, TP1G$1.C; no longer C4.+, T1G$2.C, T2.S, U1G$2.-IN
- net N$15: now also J1.TIP, VR3.3; no longer FM_ATT.3, LIN-FM.TIP
- net N$16: now also C8.1, IC2B.+IN, R12.2; no longer C6.1, R36.2, U1G$3.+IN
- net N$17: now also R5.2, VR3.2; no longer FM_ATT.2, R8.2
- net N$18: now also IC1B.OUT, TP1G$1.E, TP1G$2.E; no longer T1G$1.E, T1G$2.E, U1G$4.OUT
- net N$19: now also IC5B.-IN, R47.2; no longer R10.1, R13.2, R36.1, U1G$2.OUT
- net N$2: now also VR1.2; no longer COARSE.2
- net N$20: now also C8.2, IC2B.OUT, R8.2, T1.G; no longer C6.2, R35.2, T2.G, U1G$3.OUT
- net N$21: now also C4.1, J3.TIP; no longer C5.1, SYNC.TIP
- net N$22: now also C4.2, IC2B.-IN, R7.1, U1.CATHODE; no longer C5.2, R11.2, R12.1, U1G$3.-IN
- net N$23: now also R13.1; no longer R17.1
- net N$24: now also IC4A.-IN, R13.2, R14.1, R15.1; no longer R13.1, R14.2, R16.1, U2G$1.-IN
- net N$27: now also J6.TIP, R27.1, R29.1; no longer R24.1, R25.1, SAW.TIP
- net N$28: now also C13.2, R20.1, R23.1; no longer C7.2, R18.1, R19.1
- net N$29: now also R30.1; no longer R27.1
- net N$30: now also IC4B.-IN, R24.1, R25.2; no longer R20.1, R21.2, U2G$4.-IN
- net N$31: now also IC4B.OUT, R25.1, R27.2; no longer R21.1, R24.2, U2G$4.OUT
- net N$33: now also R23.2, R28.1; no longer R19.2, R23.1
- net N$34: now also C14.1, IC5A.-IN, R30.2, R32.2; no longer C8.1, R26.2, R27.2, U2G$3.-IN
- net N$36: now also IC3B.+IN, R18.2, R19.1; no longer R34.2, R40.1, U3G$1.+IN
- net N$37: now also C14.2, IC5A.OUT, R32.1, R33.2; no longer C8.2, R31.1, R32.2, U2G$3.OUT
- net N$39: now also IC3B.OUT, R19.2, R21.2; no longer R40.2, R41.2, U3G$1.OUT
- net N$4: now also IC1A.-IN, R3.1, TC1.1; no longer R0.1, R5.1, U1G$1.-IN
- net N$40: now also R9.1, VR4.2; no longer PWM_POT.2, R38.1
- net N$41: now also J4.TIP, VR5.3; no longer PWM.TIP, PWM_ATT.3
- net N$42: now also IC3A.-IN, R10.2, R16.1, R9.2; no longer R37.2, R38.2, R39.1, U3G$2.-IN
- net N$44: now also J5.TIP, R21.1, R22.2; no longer PULSE.TIP, R41.1, R42.2
- net N$46: now also R10.1, VR5.2; no longer PWM_ATT.2, R37.1
- net N$5: now also VR2.2; no longer FINE.2
- net N$7: now also IC1A.OUT, TC1.2; no longer R0.2, U1G$1.OUT
- net N$8: now also R6.2; no longer R4.2
- net N$9: now also J2.TIP, R3.2; no longer 1V/OCT.TIP, R5.2

Commit message: VCO 3.1
VCO Updated to V3.1 14/04/21.

Mixer section changed from Average to Sum. Mix Out is now inversion of individual outs. Might be useful?
Resistor values around mixer section reduced to 10k, inline with low noise techniques.
Parts:
- removed J1, J2, J3, J4, J5, J6, J7, J8: S_JACK, GMSN:S_JACK
- removed U1: LM4040A50IDBZT, GMSN:LM4040A50IDBZT
- removed VR1: Coarse, GMSN:9MMPOT
- removed VR2, VR3, VR4, VR5: B100K, GMSN:9MMPOT
- added 1V/OCT, LIN, MIX, PULSE, PWM_IN, SAW, SINE, SYNC, TRI: PJ301M-12, GMSN:SOCKET_MONO_3.5MMPJ301M-12
- added C20, C21: 100nF, GMSN:CAPACITOR-USC0805
- added COARSE: B100k, GMSN:RESISTOR_VARIABLEPOT_9MM_RED_KNOB
- added FINE: B100k, GMSN:RESISTOR_VARIABLEPOT_9MM_RED_MXR_KNOB
- added FM_LEVEL, PWM_LEVEL: B100k, GMSN:RESISTOR_VARIABLEPOT_9MM_GREEN_KNOB
- added IC7: TL072, GMSN:OPAMP_DUALD
- added IC8: LM4040A50IDBZT, GMSN:VOLTAGE_REF
- added PULSE_MIX, SAW_MIX, SINE_MIX, TRI_MIX: B100k, GMSN:RESISTOR_VARIABLEPOT_9MM_BLUE_KNOB
- added PULSE_WIDTH: B100k, GMSN:RESISTOR_VARIABLEPOT_9MM_YELLOW_KNOB
- added R48, R49, R50, R51, R52: 10k, GMSN:RESISTOR_USR0805
- C1, C10, C11, C12, C15, C16, C18, C19, C2, C5, C6, C9: value 100n -> 100nF; device GMSN:C-USC0805K -> GMSN:CAPACITOR-USC0805
- C13: device GMSN:C-USC0805K -> GMSN:CAPACITOR-USC0805
- C14: value 1000p -> 1nF; device GMSN:C-USC0805K -> GMSN:CAPACITOR-USC0805
- C17, C3, C4: value 100p -> 100pF; device GMSN:C-USC0805K -> GMSN:CAPACITOR-USC0805
- C7: value 2.2n -> 2.2nF; device GMSN:CAP_POLY -> GMSN:CAPACITOR_POLYFILM
- C8: value 22p -> 22pF; device GMSN:C-USC0805K -> GMSN:CAPACITOR-USC0805
- CP1, CP2: value 10u -> 10uF; device GMSN:CPOL-US153CLV-0505 -> GMSN:CAPACITOR_POL-US153CLV-0505
- D1, D2: value (none) -> STTH102A
- D3, D4: value (none) -> 1N914
- IC1, IC2, IC3, IC4, IC5, IC6: value TL072D -> TL072; device GMSN:TL072D -> GMSN:OPAMP_DUALD
- JP1: value M05X2SHD -> HEADER2X5SHD; device SparkFun-Connectors:M05X2SHD -> GMSN:HEADER2X5SHD
- R1: value 150K -> 150k; device GMSN:R-US_R0805 -> GMSN:RESISTOR_USR0805
- R10, R17: value 39K -> 39k; device GMSN:R-US_R0805 -> GMSN:RESISTOR_USR0805
- R11, R19, R2, R26, R39, R4, R6, R7: device GMSN:R-US_R0805 -> GMSN:RESISTOR_USR0805
- R12: value 9K1 -> 9k1; device GMSN:R-US_R0805 -> GMSN:RESISTOR_USR0805
- R13: value 5K6 -> 5k6; device GMSN:R-US_R0805 -> GMSN:RESISTOR_USR0805
- R14, R20, R23, R28, R38, R40, R41, R43, R44: value 10K -> 10k; device GMSN:R-US_R0805 -> GMSN:RESISTOR_USR0805
- R15: value 56K -> 56k; device GMSN:R-US_R0805 -> GMSN:RESISTOR_USR0805
- R16, R3, R30: value 100K -> 100k; device GMSN:R-US_R0805 -> GMSN:RESISTOR_USR0805
- R18: value 2K2 -> 2k2; device GMSN:R-US_R0805 -> GMSN:RESISTOR_USR0805
- R21: value 3K3 -> 1k5; device GMSN:R-US_R0805 -> GMSN:RESISTOR_USR0805
- R22: value 1K5 -> 1k5; device GMSN:R-US_R0805 -> GMSN:RESISTOR_USR0805
- R24, R25: value 22K* -> 22k; device GMSN:R-US_R0805 -> GMSN:RESISTOR_USR0805
- R27, R29, R34, R37, R42: value 2K -> 2k; device GMSN:R-US_R0805 -> GMSN:RESISTOR_USR0805
- R31: value 27K -> 27k; device GMSN:R-US_R0805 -> GMSN:RESISTOR_USR0805
- R32: value 10K -> 19k1; device GMSN:R-US_R0805 -> GMSN:RESISTOR_USR0805
- R33, R35: value 1K3 -> 1k3; device GMSN:R-US_R0805 -> GMSN:RESISTOR_USR0805
- R36, R8: value 3K3 -> 3k3; device GMSN:R-US_R0805 -> GMSN:RESISTOR_USR0805
- R45: value empty -> 100k; device GMSN:R-US_R0805 -> GMSN:RESISTOR_USR0805
- R46: value 10K -> 50k; device GMSN:R-US_R0805 -> GMSN:RESISTOR_USR0805
- R47: value 1K3 -> 0R; device GMSN:R-US_R0805 -> GMSN:RESISTOR_USR0805
- R5: value 560K -> 560k; device GMSN:R-US_R0805 -> GMSN:RESISTOR_USR0805
- R9: value 120K -> 120k; device GMSN:R-US_R0805 -> GMSN:RESISTOR_USR0805
- T1: value N_CHN -> MMBFJ309; device GMSN:N_CHN -> GMSN:TRANSISTOR_JFET_N_CHN
- TC1: value 2K -> 2k; device GMSN:R_TC -> GMSN:RESISTOR_US0207/8.5
- TP1, TP2: value TRANS_PAIR -> DMMT3904W-7-F; device GMSN:TRANS_PAIR -> GMSN:TRANSISTOR_PAIR_NPN
- TR1: device GMSN:TRIMMER_TH3 -> GMSN:RESISTOR_VARIABLETRIMMER_TH
- TR2, TR3, TR4, TR5: value 100K -> 100k; device GMSN:TRIMMER_TH3 -> GMSN:RESISTOR_VARIABLETRIMMER_TH
Connections:
- removed net N$27: J6.TIP, R27.1, R29.1
- new net N$25: IC7B.-IN, IC7B.OUT
- new net N$38: R48.1, SAW_MIX.2
- new net N$43: R49.1, TRI_MIX.2
- new net N$45: R51.1, SINE_MIX.2
- new net N$48: IC7A.-IN, R48.2, R49.2, R50.2, R51.2, R52.1
- new net N$49: IC7A.OUT, MIX.TIP, R52.2
- new net PULSE: PULSE.TIP, PULSE_MIX.3, R21.1, R22.2
- new net SAW: R27.1, R29.1, SAW.TIP, SAW_MIX.3
- net +12V: now also C20.1, COARSE.3, FINE.3, IC7P.V+, PULSE_WIDTH.3; no longer VR1.3, VR2.3, VR4.3
- net -12V: now also C21.2, COARSE.1, FINE.1, IC7P.V-, PULSE_WIDTH.1; no longer VR1.1, VR2.1, VR4.1
- net GND: now also 1V/OCT.SLEEVE, 1V/OCT.SWITCH, C20.2, C21.1, FM_LEVEL.1, IC7A.+IN, IC7B.+IN, IC8.ANODE, LIN.SLEEVE, LIN.SWITCH, MIX.SLEEVE, PULSE.SLEEVE, PULSE_MIX.1, PWM_IN.SLEEVE, PWM_LEVEL.1, SAW.SLEEVE, SAW_MIX.1, SINE.SLEEVE, SINE_MIX.1, SYNC.SLEEVE, TRI.SLEEVE, TRI_MIX.1; no longer J1.GND, J1.NORM, J2.GND, J2.NORM, J3.GND, J4.GND, J5.GND, J6.GND, J7.GND, J8.GND, U1.ANODE, VR3.1, VR5.1
- net N$15: now also FM_LEVEL.3, LIN.TIP; no longer J1.TIP, VR3.3
- net N$17: now also FM_LEVEL.2; no longer VR3.2
- net N$2: now also COARSE.2; no longer VR1.2
- net N$21: now also SYNC.TIP; no longer J3.TIP
- net N$22: now also IC8.CATHODE; no longer U1.CATHODE
- net N$40: now also PULSE_WIDTH.2; no longer VR4.2
- net N$41: now also PWM_IN.TIP, PWM_LEVEL.3; no longer J4.TIP, VR5.3
- net N$44: now also PULSE_MIX.2, R50.1; no longer J5.TIP, R21.1, R22.2
- net N$46: now also PWM_LEVEL.2; no longer VR5.2
- net N$5: now also FINE.2; no longer VR2.2
- net N$9: now also 1V/OCT.TIP; no longer J2.TIP
- net SINE: now also SINE.TIP, SINE_MIX.3; no longer J8.TIP
- net TRI: now also TRI.TIP, TRI_MIX.3; no longer J7.TIP

Commit message: Reinstall
Parts:
- removed R47: 0R, GMSN:RESISTOR_USR0805
- R7: value 87k -> 75k
Connections:
- removed net N$75: IC5B.OUT, R47.1, TR4.1, TR4.2
- net N$19: now also IC5B.OUT, TR4.1, TR4.2; no longer R47.2
Changed lines of the file:
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@@
 <part name="GND10" library="GMSN" library_urn="urn:adsk.eagle:library:27425118" deviceset="GND" device=""/>
 <part name="C4" library="GMSN" library_urn="urn:adsk.eagle:library:27425118" deviceset="CAPACITOR-US" device="C0805" package3d_urn="urn:adsk.eagle:package:27425887/1" value="100pF"/>
-<part name="R7" library="GMSN" library_urn="urn:adsk.eagle:library:27425118" deviceset="RESISTOR_US" device="R0805" package3d_urn="urn:adsk.eagle:package:27425978/1" value="87k"/>
+<part name="R7" library="GMSN" library_urn="urn:adsk.eagle:library:27425118" deviceset="RESISTOR_US" device="R0805" package3d_urn="urn:adsk.eagle:package:27425978/1" value="75k"/>
 <part name="GND9" library="GMSN" library_urn="urn:adsk.eagle:library:27425118" deviceset="GND" device=""/>
 <part name="C8" library="GMSN" library_urn="urn:adsk.eagle:library:27425118" deviceset="CAPACITOR-US" device="C0805" package3d_urn="urn:adsk.eagle:package:27425887/1" value="22pF"/>
@@
 <part name="C18" library="GMSN" library_urn="urn:adsk.eagle:library:27425118" deviceset="CAPACITOR-US" device="C0805" package3d_urn="urn:adsk.eagle:package:27425887/1" value="100nF"/>
 <part name="C19" library="GMSN" library_urn="urn:adsk.eagle:library:27425118" deviceset="CAPACITOR-US" device="C0805" package3d_urn="urn:adsk.eagle:package:27425887/1" value="100nF"/>
-<part name="R47" library="GMSN" library_urn="urn:adsk.eagle:library:27425118" deviceset="RESISTOR_US" device="R0805" package3d_urn="urn:adsk.eagle:package:27425978/1" value="0R"/>
 <part name="SAW_MIX" library="GMSN" library_urn="urn:adsk.eagle:library:27425118" deviceset="RESISTOR_VARIABLE" device="POT_9MM_BLUE_KNOB" package3d_urn="urn:adsk.eagle:package:27948773/2" value="B100k"/>
 <part name="TRI_MIX" library="GMSN" library_urn="urn:adsk.eagle:library:27425118" deviceset="RESISTOR_VARIABLE" device="POT_9MM_BLUE_KNOB" package3d_urn="urn:adsk.eagle:package:27948773/2" value="B100k"/>
@@
 <attribute name="VALUE" x="135.636" y="26.289" size="1.778" layer="96"/>
 </instance>
-<instance part="R47" gate="G$1" x="0" y="53.34" smashed="yes" rot="R180">
-<attribute name="NAME" x="3.81" y="51.8414" size="1.778" layer="95" rot="R180"/>
-<attribute name="VALUE" x="3.81" y="56.642" size="1.778" layer="96" rot="R180"/>
-</instance>
 <instance part="R45" gate="G$1" x="152.4" y="68.58" smashed="yes">
 <attribute name="NAME" x="148.59" y="70.0786" size="1.778" layer="95"/>
@@
 <wire x1="-20.32" y1="48.26" x2="-20.32" y2="60.96" width="0.1524" layer="91"/>
 <label x="-20.32" y="60.96" size="1.778" layer="95"/>
-</segment>
-</net>
-<net name="N$75" class="0">
-<segment>
-<wire x1="15.24" y1="53.34" x2="15.24" y2="40.64" width="0.1524" layer="91"/>
-<wire x1="15.24" y1="40.64" x2="17.78" y2="40.64" width="0.1524" layer="91"/>
-<wire x1="20.32" y1="40.64" x2="17.78" y2="40.64" width="0.1524" layer="91"/>
-<wire x1="17.78" y1="40.64" x2="17.78" y2="48.26" width="0.1524" layer="91"/>
-<wire x1="17.78" y1="48.26" x2="25.4" y2="48.26" width="0.1524" layer="91"/>
-<wire x1="25.4" y1="48.26" x2="25.4" y2="45.72" width="0.1524" layer="91"/>
-<junction x="17.78" y="40.64"/>
-<wire x1="15.24" y1="40.64" x2="7.62" y2="40.64" width="0.1524" layer="91"/>
-<junction x="15.24" y="40.64"/>
-<pinref part="TR4" gate="G$1" pin="1"/>
-<pinref part="TR4" gate="G$1" pin="2"/>
-<pinref part="IC5" gate="B" pin="OUT"/>
-<pinref part="R47" gate="G$1" pin="1"/>
-<wire x1="5.08" y1="53.34" x2="15.24" y2="53.34" width="0.1524" layer="91"/>
 </segment>
 </net>
@@
 <pinref part="IC5" gate="B" pin="-IN"/>
 <wire x1="-7.62" y1="43.18" x2="-15.24" y2="45.72" width="0.1524" layer="91"/>
-<pinref part="R47" gate="G$1" pin="2"/>
-<wire x1="-5.08" y1="53.34" x2="-15.24" y2="53.34" width="0.1524" layer="91"/>
-</segment>
-</net>
+<wire x1="15.24" y1="53.34" x2="15.24" y2="40.64" width="0.1524" layer="91"/>
+<wire x1="15.24" y1="40.64" x2="17.78" y2="40.64" width="0.1524" layer="91"/>
+<wire x1="20.32" y1="40.64" x2="17.78" y2="40.64" width="0.1524" layer="91"/>
+<wire x1="17.78" y1="40.64" x2="17.78" y2="48.26" width="0.1524" layer="91"/>
+<wire x1="17.78" y1="48.26" x2="25.4" y2="48.26" width="0.1524" layer="91"/>
+<wire x1="25.4" y1="48.26" x2="25.4" y2="45.72" width="0.1524" layer="91"/>
+<junction x="17.78" y="40.64"/>
+<wire x1="15.24" y1="40.64" x2="7.62" y2="40.64" width="0.1524" layer="91"/>
+<junction x="15.24" y="40.64"/>
+<pinref part="TR4" gate="G$1" pin="1"/>
+<pinref part="TR4" gate="G$1" pin="2"/>
+<pinref part="IC5" gate="B" pin="OUT"/>
+<wire x1="-15.24" y1="53.34" x2="15.24" y2="53.34" width="0.1524" layer="91"/>
+</segment>
+</net>
